File: Hardware/Flight_Controller/STM32F405_Flight_Controller_Rev2/STM32F405_Flight_Controller_Rev2.kicad_pcb (KiCad board)
At the start: 4 copper layers, 0 parts

Commit message: Ready Rev2 PCB
Parts:
- added C1: 0.1u, Capacitor_SMD:C_0603_1608Metric_Pad1.08x0.95mm_HandSolder, B.Cu at (151.4, 86.5)
- added C10: 2.2u, Capacitor_SMD:C_0603_1608Metric_Pad1.08x0.95mm_HandSolder, B.Cu at (163.8, 97.5)
- added C11: 18p, Capacitor_SMD:C_0603_1608Metric_Pad1.08x0.95mm_HandSolder, B.Cu at (150.3, 80.2)
- added C12: 18p, Capacitor_SMD:C_0603_1608Metric_Pad1.08x0.95mm_HandSolder, B.Cu at (157.0, 80.2)
- added C13: 0.1u, Capacitor_SMD:C_0603_1608Metric_Pad1.08x0.95mm_HandSolder, B.Cu at (143.9, 84.2)
- added C14: 0.1u, Capacitor_SMD:C_0603_1608Metric_Pad1.08x0.95mm_HandSolder, F.Cu at (154.4, 98.6)
- added C15: 2.2u, Capacitor_SMD:C_0603_1608Metric_Pad1.08x0.95mm_HandSolder, F.Cu at (151.4, 98.6)
- added C16: 10n, Capacitor_SMD:C_0603_1608Metric_Pad1.08x0.95mm_HandSolder, F.Cu at (151.8, 94.5)
- added C17: 0.1u, Capacitor_SMD:C_0603_1608Metric_Pad1.08x0.95mm_HandSolder, F.Cu at (147.9, 86.5)
- added C18: 0.1u, Capacitor_SMD:C_0603_1608Metric_Pad1.08x0.95mm_HandSolder, F.Cu at (145.3, 87.6)
- added C19: 1u, Capacitor_SMD:C_0603_1608Metric_Pad1.08x0.95mm_HandSolder, F.Cu at (147.2, 105.5)
- added C2: 0.1u, Capacitor_SMD:C_0603_1608Metric_Pad1.08x0.95mm_HandSolder, B.Cu at (146.6, 91.2)
- added C20: 1u, Capacitor_SMD:C_0603_1608Metric_Pad1.08x0.95mm_HandSolder, F.Cu at (147.2, 103.2)
- added C21: 0.1u, Capacitor_SMD:C_0603_1608Metric_Pad1.08x0.95mm_HandSolder, F.Cu at (160.5, 85.4)
- added C3: 0.1u, Capacitor_SMD:C_0603_1608Metric_Pad1.08x0.95mm_HandSolder, B.Cu at (150.7, 103.6)
- added C4: 0.1u, Capacitor_SMD:C_0603_1608Metric_Pad1.08x0.95mm_HandSolder, B.Cu at (163.8, 99.3)
- added C5: 0.1u, Capacitor_SMD:C_0603_1608Metric_Pad1.08x0.95mm_HandSolder, B.Cu at (162.8, 92.0)
- added C6: 4.7u, Capacitor_SMD:C_0603_1608Metric_Pad1.08x0.95mm_HandSolder, B.Cu at (148.3, 86.5)
- added C7: 0.1u, Capacitor_SMD:C_0603_1608Metric_Pad1.08x0.95mm_HandSolder, B.Cu at (157.2, 87.3)
- added C8: 1u, Capacitor_SMD:C_0603_1608Metric_Pad1.08x0.95mm_HandSolder, B.Cu at (157.2, 84.4)
- added C9: 2.2u, Capacitor_SMD:C_0603_1608Metric_Pad1.08x0.95mm_HandSolder, B.Cu at (152.6, 103.6)
- added FB1: 600R, Inductor_SMD:L_0603_1608Metric_Pad1.05x0.95mm_HandSolder, B.Cu at (161.2, 85.9)
- added H1: MountingHole_Pad, MountingHole:MountingHole_3.2mm_M3_Pad, F.Cu at (140.0, 80.0)
- added H2: MountingHole_Pad, MountingHole:MountingHole_3.2mm_M3_Pad, F.Cu at (170.0, 80.0)
- added H3: MountingHole_Pad, MountingHole:MountingHole_3.2mm_M3_Pad, F.Cu at (170.0, 110.0)
- added H4: MountingHole_Pad, MountingHole:MountingHole_3.2mm_M3_Pad, F.Cu at (140.0, 110.0)
- added J1: Conn_01x06_Socket, Connector_JST:JST_SH_SM06B-SRSS-TB_1x06-1MP_P1.00mm_Horizontal, F.Cu at (155.5, 110.1)
- added J2: Conn_01x03_Socket, Connector_JST:JST_SH_SM03B-SRSS-TB_1x03-1MP_P1.00mm_Horizontal, F.Cu at (139.8, 90.2)
- added J3: Conn_01x03_Socket, Connector_JST:JST_SH_SM03B-SRSS-TB_1x03-1MP_P1.00mm_Horizontal, F.Cu at (170.2, 98.7)
- added J4: Conn_01x03_Socket, Connector_JST:JST_SH_SM03B-SRSS-TB_1x03-1MP_P1.00mm_Horizontal, F.Cu at (170.2, 89.6)
- added J5: Conn_01x03_Socket, Connector_JST:JST_SH_SM03B-SRSS-TB_1x03-1MP_P1.00mm_Horizontal, F.Cu at (139.8, 98.5)
- added R1: 10k, Resistor_SMD:R_0603_1608Metric_Pad0.98x0.95mm_HandSolder, B.Cu at (143.8, 87.2)
- added R2: 10k, Resistor_SMD:R_0603_1608Metric_Pad0.98x0.95mm_HandSolder, B.Cu at (143.8, 88.9)
- added R3: 4.7k, Resistor_SMD:R_0603_1608Metric_Pad0.98x0.95mm_HandSolder, F.Cu at (148.0, 95.5)
- added R4: 4.7k, Resistor_SMD:R_0603_1608Metric_Pad0.98x0.95mm_HandSolder, F.Cu at (146.3, 95.5)
- added R5: 10k, Resistor_SMD:R_0603_1608Metric_Pad0.98x0.95mm_HandSolder, F.Cu at (152.7, 91.4)
- added R6: 10k, Resistor_SMD:R_0603_1608Metric_Pad0.98x0.95mm_HandSolder, F.Cu at (157.0, 81.6)
- added R7: 10k, Resistor_SMD:R_0603_1608Metric_Pad0.98x0.95mm_HandSolder, F.Cu at (147.6, 83.7)
- added TP1: TestPoint, TestPoint:TestPoint_Pad_D1.5mm, B.Cu at (138.7, 104.0)
- added TP2: TestPoint, TestPoint:TestPoint_Pad_D1.5mm, B.Cu at (141.2, 104.0)
- added TP3: TestPoint, TestPoint:TestPoint_Pad_D1.5mm, B.Cu at (143.7, 104.0)
- added TP4: TestPoint, TestPoint:TestPoint_Pad_D1.5mm, B.Cu at (146.3, 104.0)
- added U1: STM32F405RGTx, Package_QFP:LQFP-64_10x10mm_P0.5mm, B.Cu at (155.2, 95.0)
- added U2: ICM-42688-P, Sensor_Motion:ICM-42688-P, F.Cu at (155.2, 95.0)
- added U3: BMP390L, Sensor_Pressure:BMP390L, F.Cu at (147.6, 88.7)
- added U4: AP2112K-3.3, Package_TO_SOT_SMD:SOT-23-5, F.Cu at (152.0, 104.4)
- added U5: W25Q128JVS, Package_SO:SOIC-8_5.3x5.3mm_P1.27mm, F.Cu at (154.9, 86.5)
- added Y1: Crystal, Crystal:Crystal_SMD_3225-4Pin_3.2x2.5mm_HandSoldering, B.Cu at (153.7, 80.3)
Routing:
- net +3.3V: track 0.00 -> 30.0 mm
- net SPI2_MISO: track 0.00 -> 23.0 mm, vias 0 -> 1
- net GND: track 0.00 -> 18.9 mm
- net SPI2_SCK: track 0.00 -> 15.3 mm, vias 0 -> 1
- net RX6: track 0.00 -> 15.2 mm, vias 0 -> 1
- net NRST: track 0.00 -> 14.9 mm
- net TX6: track 0.00 -> 14.5 mm, vias 0 -> 1
- net SPI2_MOSI: track 0.00 -> 13.7 mm, vias 0 -> 1
- net /MCU/OSC_OUT: track 0.00 -> 13.4 mm
- net SWDIO: track 0.00 -> 11.4 mm
- net TX2: track 0.00 -> 11.2 mm, vias 0 -> 1
- net RX2: track 0.00 -> 11.1 mm, vias 0 -> 1
- net SWCLK: track 0.00 -> 10.5 mm
- net /MCU/OSC_IN: track 0.00 -> 10.4 mm
- net /MCU/BOOT0: track 0.00 -> 10.3 mm
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- added copper zone on B.Cu, net GND
- added copper zone on F.Cu, net GND
- added copper zone on In1.Cu, net GND
- added copper zone on In2.Cu, net GND
Other:
- board outline added: 38 x 38 mm
