File: Hardware/Flight_Controller/STM32F405_Flight_Controller_Rev2/STM32F405_Flight_Controller_Rev2.kicad_sch (KiCad schematic)
At the start: 0 parts

Commit message: Ready Rev2 PCB
Other:
- sheet Storage renamed Flash
- sheet Flash: file storage.kicad_sch -> flash.kicad_sch
Changed lines of the file:
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@@
 			(color 0 0 0 0)
 		)
-		(property "Sheetname" "Storage"
+		(property "Sheetname" "Flash"
 			(at 80.01 83.1084 0)
 			(show_name no)
@@
 			)
 		)
-		(property "Sheetfile" "storage.kicad_sch"
+		(property "Sheetfile" "flash.kicad_sch"
 			(at 80.01 100.9146 0)
 			(show_name no)
