File: Hardware/Flight_Controller/STM32F405_Flight_Controller_Rev2/ldo.kicad_sch (KiCad schematic)
At the start: 3 parts, among them U4 AP2112K-3.3

Commit message: Ready Rev2 PCB
Other:
- moved on the sheet: C19, C20
Changed lines of the file:
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@@
 	)
 	(junction
-		(at 134.62 91.44)
+		(at 149.86 101.6)
 		(diameter 0)
 		(color 0 0 0 0)
@@
 	)
 	(junction
-		(at 149.86 101.6)
+		(at 165.1 91.44)
 		(diameter 0)
 		(color 0 0 0 0)
 	)
 	(junction
-		(at 163.83 91.44)
+		(at 133.35 91.44)
 		(diameter 0)
 		(color 0 0 0 0)
@@
 	(wire
 		(pts
-			(xy 163.83 99.06) (xy 163.83 101.6)
-		)
-		(stroke
-			(width 0)
-			(type default)
-		)
-	)
-	(wire
-		(pts
-			(xy 157.48 91.44) (xy 163.83 91.44)
+			(xy 165.1 99.06) (xy 165.1 101.6)
+		)
+		(stroke
+			(width 0)
+			(type default)
+		)
+	)
+	(wire
+		(pts
+			(xy 157.48 91.44) (xy 165.1 91.44)
 		)
 		(stroke
@@
 	(wire
 		(pts
-			(xy 138.43 85.09) (xy 138.43 91.44)
-		)
-		(stroke
-			(width 0)
-			(type default)
-		)
-	)
-	(wire
-		(pts
-			(xy 134.62 101.6) (xy 149.86 101.6)
+			(xy 133.35 101.6) (xy 149.86 101.6)
 		)
 		(stroke
@@
 	(wire
 		(pts
-			(xy 163.83 101.6) (xy 149.86 101.6)
-		)
-		(stroke
-			(width 0)
-			(type default)
-		)
-	)
-	(wire
-		(pts
-			(xy 134.62 99.06) (xy 134.62 101.6)
-		)
-		(stroke
-			(width 0)
-			(type default)
-		)
-	)
-	(wire
-		(pts
-			(xy 134.62 91.44) (xy 138.43 91.44)
+			(xy 138.43 88.9) (xy 138.43 91.44)
+		)
+		(stroke
+			(width 0)
+			(type default)
+		)
+	)
+	(wire
+		(pts
+			(xy 133.35 91.44) (xy 138.43 91.44)
+		)
+		(stroke
+			(width 0)
+			(type default)
+		)
+	)
+	(wire
+		(pts
+			(xy 165.1 101.6) (xy 149.86 101.6)
+		)
+		(stroke
+			(width 0)
+			(type default)
+		)
+	)
+	(wire
+		(pts
+			(xy 133.35 99.06) (xy 133.35 101.6)
 		)
 		(stroke
@@
 	(symbol
 		(lib_id "power:PWR_FLAG")
-		(at 138.43 85.09 0)
+		(at 138.43 88.9 0)
 		(unit 1)
 		(body_style 1)
@@
 		(fields_autoplaced yes)
 		(property "Reference" "#FLG01"
-			(at 138.43 83.185 0)
+			(at 138.43 86.995 0)
 			(hide yes)
 			(show_name no)
@@
 		)
 		(property "Value" "PWR_FLAG"
-			(at 138.43 80.645 0)
+			(at 138.43 84.455 0)
 			(show_name no)
 			(do_not_autoplace no)
@@
 		)
 		(property "Footprint" ""
-			(at 138.43 85.09 0)
+			(at 138.43 88.9 0)
 			(hide yes)
 			(show_name no)
@@
 		)
 		(property "Datasheet" ""
-			(at 138.43 85.09 0)
+			(at 138.43 88.9 0)
 			(hide yes)
 			(show_name no)
@@
 		)
 		(property "Description" "Special symbol for telling ERC where power comes from"
-			(at 138.43 85.09 0)
+			(at 138.43 88.9 0)
 			(hide yes)
 			(show_name no)
@@
 	(symbol
 		(lib_id "Device:C")
-		(at 163.83 95.25 0)
+		(at 165.1 95.25 0)
 		(unit 1)
 		(body_style 1)
@@
 		(fields_autoplaced yes)
 		(property "Reference" "C20"
-			(at 167.64 93.9799 0)
+			(at 168.91 93.9799 0)
 			(show_name no)
 			(do_not_autoplace no)
@@
 		)
 		(property "Value" "1u"
-			(at 167.64 96.5199 0)
+			(at 168.91 96.5199 0)
 			(show_name no)
 			(do_not_autoplace no)
@@
 		)
 		(property "Footprint" "Capacitor_SMD:C_0603_1608Metric_Pad1.08x0.95mm_HandSolder"
-			(at 164.7952 99.06 0)
+			(at 166.0652 99.06 0)
 			(hide yes)
 			(show_name no)
@@
 		)
 		(property "Datasheet" ""
-			(at 163.83 95.25 0)
+			(at 165.1 95.25 0)
 			(hide yes)
 			(show_name no)
@@
 		)
 		(property "Description" "Unpolarized capacitor"
-			(at 163.83 95.25 0)
+			(at 165.1 95.25 0)
 			(hide yes)
 			(show_name no)
@@
 	(symbol
 		(lib_id "power:+3.3V")
-		(at 163.83 91.44 270)
+		(at 165.1 91.44 0)
 		(unit 1)
 		(body_style 1)
@@
 		(fields_autoplaced yes)
 		(property "Reference" "#PWR023"
-			(at 160.02 91.44 0)
+			(at 165.1 95.25 0)
 			(hide yes)
 			(show_name no)
@@
 		)
 		(property "Value" "+3.3V"
-			(at 167.005 91.4399 90)
+			(at 167.64 90.1699 0)
 			(show_name no)
 			(do_not_autoplace no)
@@
 		)
 		(property "Footprint" ""
-			(at 163.83 91.44 0)
+			(at 165.1 91.44 0)
 			(hide yes)
 			(show_name no)
@@
 		)
 		(property "Datasheet" ""
-			(at 163.83 91.44 0)
+			(at 165.1 91.44 0)
 			(hide yes)
 			(show_name no)
@@
 		)
 		(property "Description" "Power symbol creates a global label with name \"+3.3V\""
-			(at 163.83 91.44 0)
+			(at 165.1 91.44 0)
 			(hide yes)
 			(show_name no)
@@
 	(symbol
 		(lib_id "power:+5V")
-		(at 134.62 91.44 90)
+		(at 133.35 91.44 0)
+		(mirror y)
 		(unit 1)
 		(body_style 1)
@@
 		(in_pos_files yes)
 		(dnp no)
-		(fields_autoplaced yes)
 		(property "Reference" "#PWR025"
-			(at 138.43 91.44 0)
+			(at 133.35 95.25 0)
 			(hide yes)
 			(show_name no)
@@
 		)
 		(property "Value" "+5V"
-			(at 130.81 91.4399 90)
+			(at 130.81 90.1699 0)
 			(show_name no)
 			(do_not_autoplace no)
@@
 		)
 		(property "Footprint" ""
-			(at 134.62 91.44 0)
+			(at 133.35 91.44 0)
 			(hide yes)
 			(show_name no)
@@
 		)
 		(property "Datasheet" ""
-			(at 134.62 91.44 0)
+			(at 133.35 91.44 0)
 			(hide yes)
 			(show_name no)
@@
 		)
 		(property "Description" "Power symbol creates a global label with name \"+5V\""
-			(at 134.62 91.44 0)
+			(at 133.35 91.44 0)
 			(hide yes)
 			(show_name no)
@@
 	(symbol
 		(lib_id "Device:C")
-		(at 134.62 95.25 0)
+		(at 133.35 95.25 0)
 		(unit 1)
 		(body_style 1)
@@
 		(fields_autoplaced yes)
 		(property "Reference" "C19"
-			(at 138.43 93.9799 0)
+			(at 137.16 93.9799 0)
 			(show_name no)
 			(do_not_autoplace no)
@@
 		)
 		(property "Value" "1u"
-			(at 138.43 96.5199 0)
+			(at 137.16 96.5199 0)
 			(show_name no)
 			(do_not_autoplace no)
@@
 		)
 		(property "Footprint" "Capacitor_SMD:C_0603_1608Metric_Pad1.08x0.95mm_HandSolder"
-			(at 135.5852 99.06 0)
+			(at 134.3152 99.06 0)
 			(hide yes)
 			(show_name no)
@@
 		)
 		(property "Datasheet" ""
-			(at 134.62 95.25 0)
+			(at 133.35 95.25 0)
 			(hide yes)
 			(show_name no)
@@
 		)
 		(property "Description" "Unpolarized capacitor"
-			(at 134.62 95.25 0)
-			(hide yes)
-			(show_name no)
+			(at 133.35 95.25 0)
+			(hide yes)
+			(show_name no)
