File: Hardware/Flight_Controller/STM32F405_Flight_Controller_Rev2/pads_and_connectors.kicad_sch (KiCad schematic)
At the start: 11 parts, among them J1 Conn_01x06_Socket, J2 Conn_01x03_Socket, J3 Conn_01x03_Socket

Commit message: Ready Rev2 PCB
Parts:
- added J4, J5: Conn_01x03_Socket, Connector_JST:JST_SH_SM03B-SRSS-TB_1x03-1MP_P1.00mm_Horizontal, symbol Connector:Conn_01x03_Socket
Connections:
- net GND: now also J4.3 (Pin_3), J5.3 (Pin_3)
- new net RX2: J4.1 (Pin_1)
- new net RX4: J5.1 (Pin_1)
- new net TX2: J4.2 (Pin_2)
- new net TX4: J5.2 (Pin_2)
Other:
- note added: "MOTOR CONNS"
- note added: "PCB MOUNTING HOLES"
- note added: "ST-LINK PADS"
- note added: "UART1 CONN"
- note added: "UART2 CONN"
- note added: "UART4 CONN"
- note added: "UART6 CONN"
- moved on the sheet: H1, H2, H3, H4, J1, J2, J3, TP1, TP2, TP3, TP4
